File: hardware/pcb/_autosave-door-lock-pcb.kicad_sch (KiCad schematic)
At the start: 40 parts, among them J1 105162-0001, J2 Conn_01x08, J3 Conn_01x03, J4 Conn_01x04, J7 JST XH, Q1 SI2308DS, U1 ESP32-DEVKIT-V1, U2 DS1307Z+, U3 MP1470, Y1 Crystal

Commit message: progress with the PCB
Other:
- moved on the sheet: BZ1, Q1, R1
Changed lines of the file:
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@@
     (stroke (width 0) (type default))
   )
-  (wire (pts (xy 134.62 127) (xy 134.62 128.905))
+  (wire (pts (xy 133.985 122.555) (xy 133.985 124.46))
     (stroke (width 0) (type default))
   )
@@
     (stroke (width 0) (type default))
   )
-  (wire (pts (xy 134.62 135.255) (xy 134.62 133.985))
+  (wire (pts (xy 133.985 130.81) (xy 133.985 129.54))
     (stroke (width 0) (type default))
   )
@@
     (fill (type none))
   )
-  (text "5V BUCK" (at 19.05 189.23 0)
+  (text "5V BUCK" (at 19.05 191.135 0)
     (effects (font (size 3.048 3.048) (thickness 0.6096) bold) (justify left bottom))
   )
-  (text "RTC" (at 19.685 149.225 0)
+  (text "RTC" (at 19.685 150.495 0)
     (effects (font (size 3.048 3.048) (thickness 0.6096) bold) (justify left bottom))
   )
@@
     (effects (font (size 3.048 3.048) (thickness 0.6096) bold) (justify left bottom))
   )
-  (text "BUZZER" (at 107.315 150.495 0)
+  (text "BUZZER" (at 106.68 150.495 0)
     (effects (font (size 3.048 3.048) (thickness 0.6096) bold) (justify left bottom))
   )
-  (text "Mechanical" (at 118.11 189.23 0)
+  (text "Mechanical" (at 118.11 191.77 0)
     (effects (font (size 3.048 3.048) (thickness 0.6096) bold) (justify left bottom))
   )
@@
     (effects (font (size 1.27 1.27)) (justify left bottom))
   )
-  (label "BUZZER" (at 119.38 140.335 180) (fields_autoplaced)
+  (label "BUZZER" (at 118.745 135.89 180) (fields_autoplaced)
     (effects (font (size 1.27 1.27)) (justify right bottom))
   )
@@
     )
   )
-  (symbol (lib_id "Device:Buzzer") (at 137.16 131.445 0) (unit 1)
-    (in_bom yes) (on_board yes) (dnp no) (fields_autoplaced)
-    (property "Reference" "BZ1" (at 141.605 130.81 0)
-      (effects (font (size 1.27 1.27)) (justify left))
-    )
-    (property "Value" "Buzzer" (at 141.605 133.35 0)
-      (effects (font (size 1.27 1.27)) (justify left))
-    )
-    (property "Footprint" "Buzzer_Beeper:Buzzer_12x9.5RM7.6" (at 136.525 128.905 90)
-      (effects (font (size 1.27 1.27)) hide)
-    )
-    (property "Datasheet" "~" (at 136.525 128.905 90)
+  (symbol (lib_id "Device:Buzzer") (at 136.525 127 0) (unit 1)
+    (in_bom yes) (on_board yes) (dnp no) (fields_autoplaced)
+    (property "Reference" "BZ1" (at 140.97 126.365 0)
+      (effects (font (size 1.27 1.27)) (justify left))
+    )
+    (property "Value" "Buzzer" (at 140.97 128.905 0)
+      (effects (font (size 1.27 1.27)) (justify left))
+    )
+    (property "Footprint" "Buzzer_Beeper:Buzzer_12x9.5RM7.6" (at 135.89 124.46 90)
+      (effects (font (size 1.27 1.27)) hide)
+    )
+    (property "Datasheet" "~" (at 135.89 124.46 90)
       (effects (font (size 1.27 1.27)) hide)
     )
@@
     )
   )
-  (symbol (lib_id "power:GND") (at 134.62 145.415 0) (unit 1)
-    (in_bom yes) (on_board yes) (dnp no)
-    (property "Reference" "#PWR013" (at 134.62 151.765 0)
-      (effects (font (size 1.27 1.27)) hide)
-    )
-    (property "Value" "GND" (at 130.81 147.32 0)
-      (effects (font (size 1.27 1.27)))
-    )
-    (property "Footprint" "" (at 134.62 145.415 0)
-      (effects (font (size 1.27 1.27)) hide)
-    )
-    (property "Datasheet" "" (at 134.62 145.415 0)
+  (symbol (lib_id "power:GND") (at 133.985 140.97 0) (unit 1)
+    (in_bom yes) (on_board yes) (dnp no)
+    (property "Reference" "#PWR013" (at 133.985 147.32 0)
+      (effects (font (size 1.27 1.27)) hide)
+    )
+    (property "Value" "GND" (at 130.175 142.875 0)
+      (effects (font (size 1.27 1.27)))
+    )
+    (property "Footprint" "" (at 133.985 140.97 0)
+      (effects (font (size 1.27 1.27)) hide)
+    )
+    (property "Datasheet" "" (at 133.985 140.97 0)
       (effects (font (size 1.27 1.27)) hide)
     )
@@
     )
   )
-  (symbol (lib_id "Device:R") (at 123.19 140.335 90) (unit 1)
-    (in_bom yes) (on_board yes) (dnp no)
-    (property "Reference" "R1" (at 123.19 135.255 90)
-      (effects (font (size 1.27 1.27)))
-    )
-    (property "Value" "220" (at 123.19 137.795 90)
-      (effects (font (size 1.27 1.27)))
-    )
-    (property "Footprint" "Resistor_SMD:R_0805_2012Metric_Pad1.20x1.40mm_HandSolder" (at 123.19 142.113 90)
-      (effects (font (size 1.27 1.27)) hide)
-    )
-    (property "Datasheet" "~" (at 123.19 140.335 0)
+  (symbol (lib_id "Device:R") (at 122.555 135.89 90) (unit 1)
+    (in_bom yes) (on_board yes) (dnp no)
+    (property "Reference" "R1" (at 122.555 130.81 90)
+      (effects (font (size 1.27 1.27)))
+    )
+    (property "Value" "220" (at 122.555 133.35 90)
+      (effects (font (size 1.27 1.27)))
+    )
+    (property "Footprint" "Resistor_SMD:R_0805_2012Metric_Pad1.20x1.40mm_HandSolder" (at 122.555 137.668 90)
+      (effects (font (size 1.27 1.27)) hide)
+    )
+    (property "Datasheet" "~" (at 122.555 135.89 0)
       (effects (font (size 1.27 1.27)) hide)
     )
@@
     )
   )
-  (symbol (lib_id "Device:Q_NMOS_GSD") (at 132.08 140.335 0) (unit 1)
-    (in_bom yes) (on_board yes) (dnp no) (fields_autoplaced)
-    (property "Reference" "Q1" (at 138.43 139.0649 0)
-      (effects (font (size 1.27 1.27)) (justify left))
-    )
-    (property "Value" "SI2308DS" (at 138.43 141.6049 0)
-      (effects (font (size 1.27 1.27)) (justify left))
-    )
-    (property "Footprint" "Package_TO_SOT_SMD:SOT-23_Handsoldering" (at 137.16 137.795 0)
-      (effects (font (size 1.27 1.27)) hide)
-    )
-    (property "Datasheet" "~" (at 132.08 140.335 0)
+  (symbol (lib_id "Device:Q_NMOS_GSD") (at 131.445 135.89 0) (unit 1)
+    (in_bom yes) (on_board yes) (dnp no) (fields_autoplaced)
+    (property "Reference" "Q1" (at 137.795 134.6199 0)
+      (effects (font (size 1.27 1.27)) (justify left))
+    )
+    (property "Value" "SI2308DS" (at 137.795 137.1599 0)
+      (effects (font (size 1.27 1.27)) (justify left))
+    )
+    (property "Footprint" "Package_TO_SOT_SMD:SOT-23_Handsoldering" (at 136.525 133.35 0)
+      (effects (font (size 1.27 1.27)) hide)
+    )
+    (property "Datasheet" "~" (at 131.445 135.89 0)
       (effects (font (size 1.27 1.27)) hide)
     )
@@
     )
   )
-  (symbol (lib_id "power:+5V") (at 134.62 127 0) (unit 1)
-    (in_bom yes) (on_board yes) (dnp no)
-    (property "Reference" "#PWR016" (at 134.62 130.81 0)
-      (effects (font (size 1.27 1.27)) hide)
-    )
-    (property "Value" "+5V" (at 131.445 125.73 0)
-      (effects (font (size 1.27 1.27)))
-    )
-    (property "Footprint" "" (at 134.62 127 0)
-      (effects (font (size 1.27 1.27)) hide)
-    )
-    (property "Datasheet" "" (at 134.62 127 0)
-      (effects (font (size 1.27 1.27)) hide)
-    )
+  (symbol (lib_id "power:+5V") (at 133.985 122.555 0) (unit 1)
+    (in_bom yes) (on_board yes) (dnp no)
+    (property "Reference" "#PWR016" (at 133.985 126.365 0)
+      (effects (font (size 1.27 1.27)) hide)
+    )
+    (property "Value" "+5V" (at 130.81 121.285 0)
+      (effects (font (size 1.27 1.27)))
+    )
+    (property "Footprint" "" (at 133.985 122.555 0)
+      (effects (font (size 1.27 1.27)) hide)
+    )
+    (property "Datasheet" "" (at 133.985 122.555 0)
+      (effects (font (size 1.27 1.27)) hide)
+    )
