File: hardware/pcb/_autosave-door-lock-pcb.kicad_sch (KiCad schematic)
At the start: 53 parts, among them J1 105162-0001, J2 Conn_01x08, J4 Conn_01x04, J6 Conn_01x02, J7 Conn_01x02, Q1 SI2308DS, Q3 DMN6068LK3, U1 ESP32-DEVKIT-V1, U2 DS1307Z+, U3 MP1470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

Commit message: changed mosfet driver + connected sd to pwr
Parts:
- C5: now not fitted
Changed lines of the file:
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@@
   )
   (symbol (lib_id "Device:C_Polarized_Small") (at 59.69 186.69 0) (unit 1)
-    (in_bom yes) (on_board yes) (dnp no)
+    (in_bom yes) (on_board yes) (dnp yes)
     (property "Reference" "C5" (at 61.595 185.42 0)
       (effects (font (size 1.27 1.27)) (justify left))
